Commit message: Update collision meshes and materials in URDF and README
- Added new collision STL files for various links including LF, RF, LM, LR, RM, and RR components.
- Updated the README to clarify the relationship between visual and collision geometries.
- Modified the URDF to reference new collision meshes and assign appropriate material names for better visualization.

File: urdf/jumper.urdf (robot description, URDF)
Before this commit: robot jumper, 41 links, 40 joints
Links:
- link LF_finger_grip_insert_link: geometry collision mesh filename=package://kingkong_jumper_description/meshes/collision/LF_f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; visual mesh filename=package://kingkong_jumper_description/meshes/visual/LF_fing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
- link LF_finger_link: geometry collision mesh filename=package://kingkong_jumper_description/meshes/collision/LF_f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; visual mesh filename=package://kingkong_jumper_description/meshes/visual/LF_fing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
- link LF_finger_tip_link: geometry collision mesh filename=package://kingkong_jumper_description/meshes/collision/LF_f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; visual mesh filename=package://kingkong_jumper_description/meshes/visual/LF_fing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
- link LF_forearm_link: geometry collision mesh filename=package://kingkong_jumper_description/meshes/collision/LF_f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; visual mesh filename=package://kingkong_jumper_description/meshes/visual/LF_fore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
- link LF_palm_grip_insert_link: geometry collision mesh filename=package://kingkong_jumper_description/meshes/collision/LF_p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; visual mesh filename=package://kingkong_jumper_description/meshes/visual/LF_palm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
- link LF_palm_link: geometry collision mesh filename=package://kingkong_jumper_description/meshes/collision/LF_p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; visual mesh filename=package://kingkong_jumper_description/meshes/visual/LF_palm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
- link LF_palm_pad_f_link: geometry collision mesh filename=package://kingkong_jumper_description/meshes/collision/LF_p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; visual mesh filename=package://kingkong_jumper_description/meshes/visual/LF_palm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
- link LF_shoulder_link: geometry collision mesh filename=package://kingkong_jumper_description/meshes/collision/LF_s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; visual mesh filename=package://kingkong_jumper_description/meshes/visual/LF_shou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
- link LF_upper_arm_link: geometry collision mesh filename=package://kingkong_jumper_description/meshes/collision/LF_u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; visual mesh filename=package://kingkong_jumper_description/meshes/visual/LF_uppe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
- link LM_calf_link: geometry collision mesh filename=package://kingkong_jumper_description/meshes/collision/LM_c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; visual mesh filename=package://kingkong_jumper_description/meshes/visual/LM_calf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
- link LM_hip_link: geometry collision mesh filename=package://kingkong_jumper_description/meshes/collision/LM_h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; visual mesh filename=package://kingkong_jumper_description/meshes/visual/LM_hip_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
- link LM_thigh_link: geometry collision mesh filename=package://kingkong_jumper_description/meshes/collision/LM_t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; visual mesh filename=package://kingkong_jumper_description/meshes/visual/LM_thig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
- link LR_calf_link: geometry collision mesh filename=package://kingkong_jumper_description/meshes/collision/LR_c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; visual mesh filename=package://kingkong_jumper_description/meshes/visual/LR_calf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
- link LR_hip_link: geometry collision mesh filename=package://kingkong_jumper_description/meshes/collision/LR_h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; visual mesh filename=package://kingkong_jumper_description/meshes/visual/LR_hip_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
- link LR_thigh_link: geometry collision mesh filename=package://kingkong_jumper_description/meshes/collision/LR_t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; visual mesh filename=package://kingkong_jumper_description/meshes/visual/LR_thig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
- link RF_finger_grip_insert_link: geometry collision mesh filename=package://kingkong_jumper_description/meshes/collision/RF_f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; visual mesh filename=package://kingkong_jumper_description/meshes/visual/RF_fing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
- link RF_finger_link: geometry collision mesh filename=package://kingkong_jumper_description/meshes/collision/RF_f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; visual mesh filename=package://kingkong_jumper_description/meshes/visual/RF_fing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
- link RF_finger_tip_link: geometry collision mesh filename=package://kingkong_jumper_description/meshes/collision/RF_f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; visual mesh filename=package://kingkong_jumper_description/meshes/visual/RF_fing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
- link RF_forearm_link: geometry collision mesh filename=package://kingkong_jumper_description/meshes/collision/RF_f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; visual mesh filename=package://kingkong_jumper_description/meshes/visual/RF_fore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
- link RF_palm_grip_insert_link: geometry collision mesh filename=package://kingkong_jumper_description/meshes/collision/RF_p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; visual mesh filename=package://kingkong_jumper_description/meshes/visual/RF_palm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
- link RF_palm_link: geometry collision mesh filename=package://kingkong_jumper_description/meshes/collision/RF_p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; visual mesh filename=package://kingkong_jumper_description/meshes/visual/RF_palm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
- link RF_palm_pad_f_link: geometry collision mesh filename=package://kingkong_jumper_description/meshes/collision/RF_p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; visual mesh filename=package://kingkong_jumper_description/meshes/visual/RF_palm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
- link RF_shoulder_link: geometry collision mesh filename=package://kingkong_jumper_description/meshes/collision/RF_s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; visual mesh filename=package://kingkong_jumper_description/meshes/visual/RF_shou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
- link RF_upper_arm_link: geometry collision mesh filename=package://kingkong_jumper_description/meshes/collision/RF_u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; visual mesh filename=package://kingkong_jumper_description/meshes/visual/RF_uppe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
- link RM_calf_link: geometry collision mesh filename=package://kingkong_jumper_description/meshes/collision/RM_c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; visual mesh filename=package://kingkong_jumper_description/meshes/visual/RM_calf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
- link RM_hip_link: geometry collision mesh filename=package://kingkong_jumper_description/meshes/collision/RM_h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; visual mesh filename=package://kingkong_jumper_description/meshes/visual/RM_hip_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
- link RM_thigh_link: geometry collision mesh filename=package://kingkong_jumper_description/meshes/collision/RM_t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; visual mesh filename=package://kingkong_jumper_description/meshes/visual/RM_thig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
- link RR_calf_link: geometry collision mesh filename=package://kingkong_jumper_description/meshes/collision/RR_c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; visual mesh filename=package://kingkong_jumper_description/meshes/visual/RR_calf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
- link RR_hip_link: geometry collision mesh filename=package://kingkong_jumper_description/meshes/collision/RR_h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; visual mesh filename=package://kingkong_jumper_description/meshes/visual/RR_hip_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
- link RR_thigh_link: geometry collision mesh filename=package://kingkong_jumper_description/meshes/collision/RR_t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; visual mesh filename=package://kingkong_jumper_description/meshes/visual/RR_thig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
- link base_link: geometry collision mesh filename=package://kingkong_jumper_description/meshes/collision/base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; visual mesh filename=package://kingkong_jumper_description/meshes/visual/base_li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
- link camera_link: geometry collision mesh filename=package://kingkong_jumper_description/meshes/collision/came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; visual mesh filename=package://kingkong_jumper_description/meshes/visual/camera_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
- link display_module_link: geometry collision mesh filename=package://kingkong_jumper_description/meshes/collision/disp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; visual mesh filename=package://kingkong_jumper_description/meshes/visual/display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
- link tof_sensor_link: geometry collision mesh filename=package://kingkong_jumper_description/meshes/collision/tof_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; visual mesh filename=package://kingkong_jumper_description/meshes/visual/tof_sen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
- link upper_shell_link: geometry collision mesh filename=package://kingkong_jumper_description/meshes/collision/uppe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; visual mesh filename=package://kingkong_jumper_description/meshes/visual/upper_s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
